File: eagle/9volt_power_rail/9volt_rail.sch (EAGLE design)
At the start: 32 parts, among them X1 5566-4, X2 5566-4, X3 5566-4, X4 5566-4, X5 5566-4, X6 5566-4

Commit message: working on width errors
Parts:
- removed C1, C5, C7: 330uF, rcl:CPOL-USE5-10.5
- removed C2, C6, C8: 2.2uF, adafruit:C-USC0805
- removed JP1: (no value), adafruit:PINHD-1X12
- removed R1, R10, R7: (no value), adafruit:R-US_M0805
- removed U$1, U$5, U$7: PTH78020-SMD, PTN78020:PTH78020-SMD
- removed U$2, U$6, U$8: 3310-001, 3310-001:3310-001
- removed X1, X2, X3, X4, X5, X6: 5566-4, con-molex:5566-4
- added PL1, PL10, PL12, PL2, PL3, PL4, PL5, PL6, PL7, PL8, PL9: (no value), con-molex-2:555X-2H
- added PL11: (no value), con-molex-2:555X-4H
- renumbered LED1 to VCC
Connections:
- removed net N$10: JP1.7, JP1.8, X6-1.S, X6-2.S
- removed net N$17: U$5.ADJ, U$6.TWO
- removed net N$2: U$1.ADJ, U$2.TWO
- removed net N$22: U$7.ADJ, U$8.TWO
- removed net N$3: C1.+, R1.1, U$1.SEN, U$1.VOUT, X1-4.S
- removed net N$6: C5.+, R7.1, U$5.SEN, U$5.VOUT, X4-3.S, X4-4.S
- removed net N$7: JP1.5, JP1.6, X6-3.S, X6-4.S
- removed net N$9: C7.+, R10.1, U$7.SEN, U$7.VOUT, X5-3.S, X5-4.S
- net GND: now also PL1-1.S, PL10-1.S, PL11-1.S, PL11-2.S, PL12-1.S, PL2-1.S, PL3-1.S, PL4-1.S, PL5-1.S, PL6-1.S, PL7-1.S, PL8-1.S, PL9-1.S; no longer C1.-, C2.2, C5.-, C6.2, C7.-, C8.2, JP1.3, JP1.4, R1.2, R10.2, R7.2, U$1.GND1, U$1.GND2, U$2.THREE, U$5.GND1, U$5.GND2, U$6.THREE, U$7.GND1, U$7.GND2, U$8.THREE, X1-2.S, X2-2.S, X3-1.S, X3-2.S, X4-1.S, X4-2.S, X5-1.S, X5-2.S
- net N$1: now also PL1-2.S, PL10-2.S, PL11-3.S, PL11-4.S, PL2-2.S, PL3-2.S, PL4-2.S, PL5-2.S, PL6-2.S, PL7-2.S, PL8-2.S, PL9-2.S; no longer X2-4.S
- net N$5: no longer JP1.9, U$1.INH, U$5.INH, U$7.INH
- net VCC: now also PL12-2.S; no longer C2.1, C6.1, C8.1, JP1.1, JP1.2, U$1.VIN, U$5.VIN, U$7.VIN, X3-3.S, X3-4.S

Commit message: Done with revision B
Parts:
- removed VCC: (no value), adafruit:LED5MM
- added IC1: TL331, linear:TL331
- added JP1: (no value), adafruit:PINHD-1X3
- added PL13: (no value), con-molex-2:555X-4H
- added R1, R10, R11, R3, R5, R7: (no value), adafruit:R-US_M0805
- added R6: (no value), pot:TRIM_US-RS3
- added T1: (no value), zetex:PMOSSOT223
- added VCC1, VCC2, VCC3: (no value), adafruit:LED5MM
Connections:
- removed net N$14: R8.2, R9.1, T3.G
- new net N$10: R11.1, T1.S
- new net N$2: IC1.OUT, JP1.1, JP1.2, JP1.3, R8.1, R9.2, T1.G, T3.G
- new net N$3: R1.2, R5.1, VCC1.A
- new net N$6: R2.1, R3.2, R6.E
- new net N$7: IC1.-IN, R5.2, R7.1
- new net N$8: R11.2, VCC3.A
- new net N$9: R4.2, VCC2.A
- net GND: now also IC1.GND, PL13-1.S, PL13-2.S, R10.2, R6.S, R7.2, VCC1.C, VCC2.C, VCC3.C; no longer R4.2, R9.2
- net N$1: now also PL13-3.S, PL13-4.S, R10.1
- net N$4: now also IC1.+IN, R2.2, R9.1; no longer R2.1, VCC.C
- net N$5: no longer R2.2
- net VCC: now also IC1.V+, R1.1, R3.1, R8.2, T1.D; no longer R8.1, VCC.A
Other:
- moved on the sheet: PL12-1, PL12-2, R2, R8, R9, T3
