File: eagle/9volt_power_rail/9volt_rail.sch (EAGLE design)
At the start: 48 parts, among them IC1 TL331

Commit message: Done with power board and adc cape
Parts:
- removed T1, T3: (no value), zetex:PMOSSOT223
- added H1, H2, H3, H4: MOUNT-PAD-ROUND3.0, holes:MOUNT-PAD-ROUND3.0
- added Q1: BSS84, transistor-small-signal:BSS84
- added Q2: BSS123, transistor-small-signal:BSS123
- added R12: (no value), adafruit:R-US_M0805
Connections:
- net GND: now also H1.MOUNT, H2.MOUNT, H3.MOUNT, H4.MOUNT, Q2.S, R12.2; no longer T3.D
- net N$10: now also Q2.D, U$3.INH; no longer R11.1, T1.D
- net N$2: now also Q1.G; no longer T1.G, T3.G
- net N$5: now also Q1.D, Q2.G, R11.1, R12.1; no longer T3.S, U$3.INH
- net VCC: now also Q1.S; no longer T1.S
Changed lines of the file:
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@@
 <part name="U$4" library="3310-001" deviceset="3310-001" device=""/>
 <part name="GND8" library="supply1" deviceset="GND" device=""/>
-<part name="T3" library="zetex" deviceset="PMOSSOT223" device=""/>
 <part name="GND17" library="supply1" deviceset="GND" device=""/>
 <part name="P+4" library="supply1" deviceset="VCC" device=""/>
@@
 <part name="R10" library="adafruit" deviceset="R-US_" device="M0805"/>
 <part name="VCC2" library="adafruit" deviceset="LED" device="5MM"/>
-<part name="T1" library="zetex" deviceset="PMOSSOT223" device=""/>
 <part name="VCC3" library="adafruit" deviceset="LED" device="5MM"/>
 <part name="R11" library="adafruit" deviceset="R-US_" device="M0805"/>
@@
 <part name="C14" library="adafruit" deviceset="C-US" device="C0805" value="2.2uF"/>
 <part name="C15" library="adafruit" deviceset="C-US" device="C0805" value="2.2uF"/>
+<part name="H1" library="holes" deviceset="MOUNT-PAD-ROUND" device="3.0"/>
+<part name="H2" library="holes" deviceset="MOUNT-PAD-ROUND" device="3.0"/>
+<part name="H3" library="holes" deviceset="MOUNT-PAD-ROUND" device="3.0"/>
+<part name="H4" library="holes" deviceset="MOUNT-PAD-ROUND" device="3.0"/>
+<part name="R12" library="adafruit" deviceset="R-US_" device="M0805"/>
+<part name="Q1" library="transistor-small-signal" deviceset="BSS84" device=""/>
+<part name="Q2" library="transistor-small-signal" deviceset="BSS123" device=""/>
 </parts>
 <sheets>
@@
 <instance part="U$4" gate="G$1" x="66.04" y="-25.4"/>
 <instance part="GND8" gate="1" x="53.34" y="-48.26"/>
-<instance part="T3" gate="G$1" x="40.64" y="-48.26" rot="R180"/>
 <instance part="GND17" gate="1" x="40.64" y="-83.82"/>
 <instance part="P+4" gate="VCC" x="20.32" y="20.32"/>
@@
 <instance part="R10" gate="G$1" x="109.22" y="0" rot="R270"/>
 <instance part="VCC2" gate="G$1" x="96.52" y="-17.78"/>
-<instance part="T1" gate="G$1" x="0" y="12.7" rot="R180"/>
 <instance part="VCC3" gate="G$1" x="0" y="-35.56"/>
 <instance part="R11" gate="G$1" x="0" y="-15.24" rot="R270"/>
@@
 <instance part="C14" gate="G$1" x="27.94" y="2.54"/>
 <instance part="C15" gate="G$1" x="35.56" y="2.54"/>
+<instance part="H1" gate="G$1" x="-139.7" y="-27.94"/>
+<instance part="H2" gate="G$1" x="-139.7" y="-35.56"/>
+<instance part="H3" gate="G$1" x="-139.7" y="-43.18"/>
+<instance part="H4" gate="G$1" x="-139.7" y="-50.8"/>
+<instance part="R12" gate="G$1" x="10.16" y="-15.24" rot="R270"/>
+<instance part="Q1" gate="G$1" x="0" y="12.7"/>
+<instance part="Q2" gate="G$1" x="40.64" y="-35.56"/>
 </instances>
 <busses>
@@
 <wire x1="-40.64" y1="-78.74" x2="-22.86" y2="-78.74" width="0.1524" layer="91"/>
 <wire x1="-22.86" y1="-78.74" x2="0" y2="-78.74" width="0.1524" layer="91"/>
-<wire x1="0" y1="-78.74" x2="40.64" y2="-78.74" width="0.1524" layer="91"/>
+<wire x1="0" y1="-78.74" x2="10.16" y2="-78.74" width="0.1524" layer="91"/>
+<wire x1="10.16" y1="-78.74" x2="40.64" y2="-78.74" width="0.1524" layer="91"/>
 <wire x1="-91.44" y1="-78.74" x2="-63.5" y2="-78.74" width="0.1524" layer="91"/>
 <junction x="-40.64" y="-78.74"/>
@@
 <wire x1="0" y1="-40.64" x2="0" y2="-78.74" width="0.1524" layer="91"/>
 <junction x="0" y="-78.74"/>
-<pinref part="T3" gate="G$1" pin="D"/>
-<wire x1="40.64" y1="-53.34" x2="40.64" y2="-78.74" width="0.1524" layer="91"/>
+<pinref part="R12" gate="G$1" pin="2"/>
+<wire x1="10.16" y1="-20.32" x2="10.16" y2="-78.74" width="0.1524" layer="91"/>
+<junction x="10.16" y="-78.74"/>
+<wire x1="40.64" y1="-43.18" x2="40.64" y2="-45.72" width="0.1524" layer="91"/>
 <junction x="40.64" y="-78.74"/>
+<pinref part="Q2" gate="G$1" pin="S"/>
+<wire x1="40.64" y1="-45.72" x2="40.64" y2="-78.74" width="0.1524" layer="91"/>
+<wire x1="40.64" y1="-40.64" x2="40.64" y2="-43.18" width="0.1524" layer="91"/>
 </segment>
 <segment>
@@
 <pinref part="GND18" gate="1" pin="GND"/>
 <wire x1="-114.3" y1="2.54" x2="-106.68" y2="2.54" width="0.1524" layer="91"/>
-<wire x1="-106.68" y1="2.54" x2="-106.68" y2="-17.78" width="0.1524" layer="91"/>
+<wire x1="-106.68" y1="2.54" x2="-106.68" y2="-12.7" width="0.1524" layer="91"/>
+<wire x1="-106.68" y1="-12.7" x2="-106.68" y2="-17.78" width="0.1524" layer="91"/>
+<wire x1="-106.68" y1="-12.7" x2="-144.78" y2="-12.7" width="0.1524" layer="91"/>
+<junction x="-106.68" y="-12.7"/>
+<pinref part="H1" gate="G$1" pin="MOUNT"/>
+<wire x1="-142.24" y1="-27.94" x2="-144.78" y2="-27.94" width="0.1524" layer="91"/>
+<wire x1="-144.78" y1="-27.94" x2="-144.78" y2="-12.7" width="0.1524" layer="91"/>
+<pinref part="H2" gate="G$1" pin="MOUNT"/>
+<wire x1="-142.24" y1="-35.56" x2="-144.78" y2="-35.56" width="0.1524" layer="91"/>
+<wire x1="-144.78" y1="-35.56" x2="-144.78" y2="-27.94" width="0.1524" layer="91"/>
+<junction x="-144.78" y="-27.94"/>
+<pinref part="H3" gate="G$1" pin="MOUNT"/>
+<wire x1="-142.24" y1="-43.18" x2="-144.78" y2="-43.18" width="0.1524" layer="91"/>
+<wire x1="-144.78" y1="-43.18" x2="-144.78" y2="-35.56" width="0.1524" layer="91"/>
+<junction x="-144.78" y="-35.56"/>
+<pinref part="H4" gate="G$1" pin="MOUNT"/>
+<wire x1="-142.24" y1="-50.8" x2="-144.78" y2="-50.8" width="0.1524" layer="91"/>
+<wire x1="-144.78" y1="-50.8" x2="-144.78" y2="-43.18" width="0.1524" layer="91"/>
+<junction x="-144.78" y="-43.18"/>
 </segment>
 <segment>
@@
 <net name="N$5" class="0">
 <segment>
-<pinref part="U$3" gate="G$1" pin="INH"/>
-<wire x1="40.64" y1="-25.4" x2="50.8" y2="-25.4" width="0.1524" layer="91"/>
-<wire x1="50.8" y1="-25.4" x2="50.8" y2="-5.08" width="0.1524" layer="91"/>
-<pinref part="T3" gate="G$1" pin="S"/>
-<wire x1="40.64" y1="-43.18" x2="40.64" y2="-25.4" width="0.1524" layer="91"/>
+<pinref part="R11" gate="G$1" pin="1"/>
+<wire x1="0" y1="7.62" x2="0" y2="-7.62" width="0.1524" layer="91"/>
+<pinref part="R12" gate="G$1" pin="1"/>
+<wire x1="0" y1="-7.62" x2="0" y2="-10.16" width="0.1524" layer="91"/>
+<wire x1="10.16" y1="-10.16" x2="10.16" y2="-7.62" width="0.1524" layer="91"/>
+<wire x1="10.16" y1="-7.62" x2="0" y2="-7.62" width="0.1524" layer="91"/>
+<junction x="0" y="-7.62"/>
+<pinref part="Q1" gate="G$1" pin="D"/>
+<pinref part="Q2" gate="G$1" pin="G"/>
+<wire x1="35.56" y1="-38.1" x2="15.24" y2="-38.1" width="0.1524" layer="91"/>
+<wire x1="15.24" y1="-38.1" x2="15.24" y2="-7.62" width="0.1524" layer="91"/>
+<wire x1="15.24" y1="-7.62" x2="10.16" y2="-7.62" width="0.1524" layer="91"/>
+<junction x="10.16" y="-7.62"/>
 </segment>
 </net>
@@
 <wire x1="0" y1="25.4" x2="-15.24" y2="25.4" width="0.1524" layer="91"/>
 <junction x="-15.24" y="25.4"/>
-<pinref part="T1" gate="G$1" pin="S"/>
 <wire x1="0" y1="17.78" x2="0" y2="25.4" width="0.1524" layer="91"/>
+<pinref part="Q1" gate="G$1" pin="S"/>
 </segment>
 </net>
@@
 <pinref part="IC1" gate="G$1" pin="OUT"/>
 <pinref part="R8" gate="G$1" pin="1"/>
-<wire x1="15.24" y1="-50.8" x2="-7.62" y2="-50.8" width="0.1524" layer="91"/>
-<wire x1="-7.62" y1="-50.8" x2="-15.24" y2="-50.8" width="0.1524" layer="91"/>
+<wire x1="15.24" y1="-50.8" x2="-10.16" y2="-50.8" width="0.1524" layer="91"/>
+<wire x1="-10.16" y1="-50.8" x2="-15.24" y2="-50.8" width="0.1524" layer="91"/>
 <wire x1="-15.24" y1="-50.8" x2="-22.86" y2="-50.8" width="0.1524" layer="91"/>
 <wire x1="-22.86" y1="-50.8" x2="-33.02" y2="-50.8" width="0.1524" layer="91"/>
@@
 <wire x1="-22.86" y1="-38.1" x2="-22.86" y2="-50.8" width="0.1524" layer="91"/>
 <junction x="-22.86" y="-50.8"/>
-<wire x1="-7.62" y1="17.78" x2="-7.62" y2="-50.8" width="0.1524" layer="91"/>
-<junction x="-7.62" y="-50.8"/>
 <wire x1="15.24" y1="-50.8" x2="15.24" y2="-60.96" width="0.1524" layer="91"/>
 <pinref part="JP1" gate="A" pin="1"/>
@@
 <wire x1="15.24" y1="-66.04" x2="15.24" y2="-63.5" width="0.1524" layer="91"/>
 <junction x="15.24" y="-63.5"/>
-<wire x1="-7.62" y1="17.78" x2="7.62" y2="17.78" width="0.1524" layer="91"/>
-<wire x1="7.62" y1="17.78" x2="7.62" y2="15.24" width="0.1524" layer="91"/>
-<pinref part="T1" gate="G$1" pin="G"/>
-<wire x1="7.62" y1="15.24" x2="5.08" y2="15.24" width="0.1524" layer="91"/>
-<pinref part="T3" gate="G$1" pin="G"/>
-<wire x1="45.72" y1="-45.72" x2="48.26" y2="-45.72" width="0.1524" layer="91"/>
-<wire x1="48.26" y1="-45.72" x2="48.26" y2="-43.18" width="0.1524" layer="91"/>
-<wire x1="48.26" y1="-43.18" x2="33.02" y2="-43.18" width="0.1524" layer="91"/>
-<wire x1="33.02" y1="-43.18" x2="33.02" y2="-50.8" width="0.1524" layer="91"/>
-<wire x1="33.02" y1="-50.8" x2="15.24" y2="-50.8" width="0.1524" layer="91"/>
-<junction x="15.24" y="-50.8"/>
+<pinref part="Q1" gate="G$1" pin="G"/>
+<wire x1="-5.08" y1="15.24" x2="-10.16" y2="15.24" width="0.1524" layer="91"/>
+<wire x1="-10.16" y1="15.24" x2="-10.16" y2="-50.8" width="0.1524" layer="91"/>
+<junction x="-10.16" y="-50.8"/>
 </segment>
 </net>
@@
 <net name="N$10" class="0">
 <segment>
-<pinref part="T1" gate="G$1" pin="D"/>
-<pinref part="R11" gate="G$1" pin="1"/>
-<wire x1="0" y1="7.62" x2="0" y2="-10.16" width="0.1524" layer="91"/>
-</segment>
-</net>
+<pinref part="U$3" gate="G$1" pin="INH"/>
+<wire x1="50.8" y1="-25.4" x2="50.8" y2="-5.08" width="0.1524" layer="91"/>
+<wire x1="40.64" y1="-25.4" x2="50.8" y2="-25.4" width="0.1524" layer="91"/>
+<pinref part="Q2" gate="G$1" pin="D"/>
+<wire x1="40.64" y1="-25.4" x2="40.64" y2="-30.48" width="0.1524" layer="91"/>
+</segment>
+</net>

Commit message: update to adc cape
Other:
- moved on the sheet: C11, C12, C13, C14, C15, C4
