File: eagle/ADC_Board/adc_cap.brd (EAGLE design)
At the start: 97.5 x 56.5 mm, 38 parts, among them Q1 BSS84, Q2 BSS84, Q3 BSS84, Q4 BSS84, Q5 BSS84, Q6 BSS84, Q7 BSS84, Q8 BSS84, X1 53048-11, X10 53048-11, X11 53048-11, X5 53048-11, X6 53048-11, X7 53048-11, X8 53048-11, X9 53048-11

Commit message: Done with power board and adc cape
Parts:
- added C1, C10, C11, C12, C13, C14, C15, C16, C17, C2, C3, C4, C5, C6, C7, C8, C9: (no value), rcl:C0805
- added R11, R14, R15, R16: (no value), rcl:R0805
- moved PL1 0.95 mm to (8.57, 27.0)
Connections:
- removed net VDD_3V3EXP: U$1.181, U$1.182
- new net N$80: R11.2, U$1.167
- new net N$81: R15.1, U$1.165
- new net N$85: R14.2, U$1.168
- new net N$86: R16.1, U$1.166
- new net N$88: C17.1, R12.1, R13.1, R6.2, U$1.181, U$1.182
- net GND: now also C1.2, C10.2, C11.2, C12.2, C13.2, C14.2, C15.2, C16.2, C17.2, C2.2, C3.2, C4.2, C5.2, C6.2, C7.2, C8.2, C9.2
- net N$55: now also R14.1, R16.2; no longer U$1.168
- net N$75: now also C4.1
- net N$76: now also C3.1
- net N$77: now also C1.1
- net N$78: now also C7.1
- net N$79: now also C2.1
- net N$82: now also C5.1
- net N$83: now also C8.1
- net N$84: now also R11.1, R15.2; no longer U$1.165
- net N$87: now also C6.1
- net VCC: now also C10.1, C11.1, C12.1, C13.1, C14.1, C15.1, C16.1, C9.1; no longer R12.1, R13.1, R6.2
Routing:
- net N$88: track 0.00 -> 65.1 mm, vias 0 -> 1
- net N$80: track 0.00 -> 18.8 mm
- net N$86: track 0.00 -> 14.8 mm
- net VCC: track 380.3 -> 389.5 mm
- net N$85: track 0.00 -> 8.23 mm
- net N$83: track 8.67 -> 16.6 mm
- net N$81: track 0.00 -> 7.03 mm
- net N$84: track 200.1 -> 193.9 mm
- net N$82: track 5.54 -> 11.6 mm
- net N$76: track 6.11 -> 10.9 mm
- net N$77: track 8.42 -> 12.3 mm
- net N$78: track 7.31 -> 11.1 mm
- net N$55: track 183.1 -> 180.3 mm
- net N$87: track 6.55 -> 9.33 mm
- net N$75: track 6.48 -> 9.22 mm
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Other:
- board size 97.5 x 56.5 mm -> 97.5 x 56.2 mm
