File: eagle/ADC_Board/adc_cap.sch (EAGLE design)
At the start: 38 parts, among them Q1 BSS84, Q2 BSS84, Q3 BSS84, Q4 BSS84, Q5 BSS84, Q6 BSS84, Q7 BSS84, Q8 BSS84, X1 53048-11, X10 53048-11, X11 53048-11, X5 53048-11, X6 53048-11, X7 53048-11, X8 53048-11, X9 53048-11

Commit message: Done with power board and adc cape
Parts:
- added C1, C10, C11, C12, C13, C14, C15, C16, C17, C2, C3, C4, C5, C6, C7, C8, C9: (no value), rcl:C-USC0805
- added R11, R14, R15, R16: (no value), rcl:R-US_R0805
Connections:
- new net N$80: R11.2, U$1.I2C2_SDA
- new net N$81: R15.1, U$1.I2C1_SDA
- new net N$85: R14.2, U$1.I2C1_SCL
- new net N$86: R16.1, U$1.I2C2_SCL
- new net N$88: C17.1, R12.1, R13.1, R6.2, U$1.VDD_3V3EXP@1, U$1.VDD_3V3EXP@2
- net GND: now also C1.2, C10.2, C11.2, C12.2, C13.2, C14.2, C15.2, C16.2, C17.2, C2.2, C3.2, C4.2, C5.2, C6.2, C7.2, C8.2, C9.2
- net N$55: now also R14.1, R16.2; no longer U$1.I2C1_SCL
- net N$75: now also C4.1
- net N$76: now also C3.1
- net N$77: now also C1.1
- net N$78: now also C7.1
- net N$79: now also C2.1
- net N$82: now also C5.1
- net N$83: now also C8.1
- net N$84: now also R11.1, R15.2; no longer U$1.I2C1_SDA
- net N$87: now also C6.1
- net VCC: now also C10.1, C11.1, C12.1, C13.1, C14.1, C15.1, C16.1, C9.1; no longer R12.1, R13.1, R6.2
Other:
- moved on the sheet: U$1
